File: ringmod.kicad_pcb (KiCad board)
At the start: 2 copper layers, 64.5 x 39.9 mm, 21 parts, among them P1 CONN_01X01, P2 CONN_01X01, P3 CONN_01X01, P4 CONN_01X01, P5 CONN_01X01, P6 CONN_01X01, T1 audio_transformer, T2 audio_transformer

Commit message: fix schematic and enlarge mechanical holes for the transformers
Parts:
- T1, T2: footprint trafo-xicon:trafo-xicon-42TM -> ringmod:trafo-xicon-42TM
- moved D3 10.5 mm to (147.2, 83.5), turned to 315 degrees
- moved D1 10.3 mm to (153.8, 99.2), turned to 225 degrees
- moved D2 9.80 mm to (139.8, 106.5), turned to 135 degrees
- moved D4 9.65 mm to (132.5, 90.8), turned to 45 degrees
Connections:
- D2 pad 1: Net-(D2-Pad1) -> Net-(D1-Pad2)
- D2 pad 2: Net-(D1-Pad1) -> Net-(D2-Pad2)
- D3 pad 1: Net-(D1-Pad2) -> Net-(D3-Pad1)
- D3 pad 2: Net-(D3-Pad2) -> Net-(D1-Pad1)
- D4 pad 1: Net-(D3-Pad2) -> Net-(D2-Pad2)
- D4 pad 2: Net-(D2-Pad1) -> Net-(D3-Pad1)
- T1 pad 1: Net-(D3-Pad2) -> Net-(D3-Pad1)
- T1 pad 3: Net-(D1-Pad1) -> Net-(D1-Pad2)
- T2 pad 1: Net-(D1-Pad2) -> Net-(D1-Pad1)
- T2 pad 3: Net-(D2-Pad1) -> Net-(D2-Pad2)
Routing:
- net Net-(D3-Pad2): track 25.1 -> 0.00 mm
- net Net-(D3-Pad1): track 0.00 -> 25.1 mm
- net Net-(D1-Pad2): track 42.4 -> 24.7 mm
- net Net-(D1-Pad1): track 24.7 -> 42.4 mm
- net Net-(D2-Pad2): track 0.00 -> 15.7 mm
- net Net-(D2-Pad1): track 15.7 -> 0.00 mm
